Commit message: Moved the camera sensor down to a lower height for the SensorBox project.

File: interbotix_ros_xslocobots/interbotix_xslocobot_descriptions/urdf/locobot.urdf.xacro (robot description, xacro)
@@ -339,5 +339,8 @@
     <limit effort="2" lower="${-pi/2}" upper="${pi/2}" velocity="${pi}"/>
     <xacro:if value="${arm_type == 'mobile_wx250s'}">
+    <!-- TODO-JYW:
       <origin rpy="0 0 0" xyz="0.047228 0 0.44425"/>
+      -->
+      <origin rpy="0 0 0" xyz="0.047228 0 0.05200"/>
     </xacro:if>
     <xacro:unless value="${arm_type == 'mobile_wx250s'}">

Commit message: Modifying the base_footprint diameter to allow navigation in a more cluttererd environment.

File: interbotix_ros_xslocobots/interbotix_xslocobot_descriptions/urdf/locobot.urdf.xacro (robot description, xacro)
@@ -38,5 +38,7 @@
       <origin rpy="0 0 0" xyz="0.0 0 0.05949"/>
       <geometry>
-        <cylinder length="0.10938" radius="0.178"/>
+	      <!-- TODO-JYW: Reducing the radius by half to determine if this affects the proximity to obstacles. -->
+	      <!-- <cylinder length="0.10938" radius="0.178"/> -->
+        <cylinder length="0.10938" radius="0.089"/>
       </geometry>
     </collision>
